Commit message: feat: adding test axol ik

File: assets/axol/urdf/axol.urdf (robot description, URDF)
Before this commit: robot assembly, 19 links, 18 joints
Links:
- link base: geometry collision mesh filename=meshes/Base.stl scale=1 1 1; visual mesh filename=meshes/Base.stl scale=1 1 1
- link left_e1: geometry collision mesh filename=meshes/Left_E1.stl scale=1 1 1; visual mesh filename=meshes/Left_E1.stl scale=1 1 1
- link left_e2: geometry collision mesh filename=meshes/Left_E2.stl scale=1 1 1; visual mesh filename=meshes/Left_E2.stl scale=1 1 1
- link left_gripper: geometry collision mesh filename=meshes/Left_Gripper.stl scale=1 1 1; visual mesh filename=meshes/Left_Gripper.stl scale=1 1 1
- link left_s2: geometry collision mesh filename=meshes/Left_S2.stl scale=1 1 1; visual mesh filename=meshes/Left_S2.stl scale=1 1 1
- link left_s3: geometry collision mesh filename=meshes/Left_S3.stl scale=1 1 1; visual mesh filename=meshes/Left_S3.stl scale=1 1 1
- link left_w0: geometry collision mesh filename=meshes/Left_W0.stl scale=1 1 1; visual mesh filename=meshes/Left_W0.stl scale=1 1 1
- link left_w1: geometry collision mesh filename=meshes/Left_W1.stl scale=1 1 1; visual mesh filename=meshes/Left_W1.stl scale=1 1 1
- link left_w2: geometry collision mesh filename=meshes/Left_W2.stl scale=1 1 1; visual mesh filename=meshes/Left_W2.stl scale=1 1 1
- link right_e1: geometry collision mesh filename=meshes/Right_E1.stl scale=1 1 1; visual mesh filename=meshes/Right_E1.stl scale=1 1 1
- link right_e2: geometry collision mesh filename=meshes/Right_E2.stl scale=1 1 1; visual mesh filename=meshes/Right_E2.stl scale=1 1 1
- link right_gripper: geometry collision mesh filename=meshes/Right_Gripper.stl scale=1 1 1; visual mesh filename=meshes/Right_Gripper.stl scale=1 1 1
- link right_s2: geometry collision mesh filename=meshes/Right_S2.stl scale=1 1 1; visual mesh filename=meshes/Right_S2.stl scale=1 1 1
- link right_s3: geometry collision mesh filename=meshes/Right_S3.stl scale=1 1 1; visual mesh filename=meshes/Right_S3.stl scale=1 1 1
- link right_w0: geometry collision mesh filename=meshes/Right_W0.stl scale=1 1 1; visual mesh filename=meshes/Right_W0.stl scale=1 1 1
- link right_w1: geometry collision mesh filename=meshes/Right_W1.stl scale=1 1 1; visual mesh filename=meshes/Right_W1.stl scale=1 1 1
- link right_w2: geometry collision mesh filename=meshes/Right_W2.stl scale=1 1 1; visual mesh filename=meshes/Right_W2.stl scale=1 1 1
- link s1: geometry collision mesh filename=meshes/S1.stl scale=1 1 1; visual mesh filename=meshes/S1.stl scale=1 1 1

Commit message: feat: pulling mitshell ik solver

File: assets/axol/urdf/axol.urdf (robot description, URDF)
Before this commit: robot assembly, 19 links, 18 joints
Links:
- link base: geometry collision mesh filename=package://assembly/meshes/Base.stl scale=1 1 1; visual mesh filename=package://assembly/meshes/Base.stl scale=1 1 1
- link left_e1: geometry collision mesh filename=package://assembly/meshes/Left_E1.stl scale=1 1 1; visual mesh filename=package://assembly/meshes/Left_E1.stl scale=1 1 1
- link left_e2: geometry collision mesh filename=package://assembly/meshes/Left_E2.stl scale=1 1 1; visual mesh filename=package://assembly/meshes/Left_E2.stl scale=1 1 1
- link left_gripper: geometry collision mesh filename=package://assembly/meshes/Left_Gripper.stl scale=1 1 1; visual mesh filename=package://assembly/meshes/Left_Gripper.stl scale=1 1 1
- link left_s2: geometry collision mesh filename=package://assembly/meshes/Left_S2.stl scale=1 1 1; visual mesh filename=package://assembly/meshes/Left_S2.stl scale=1 1 1
- link left_s3: geometry collision mesh filename=package://assembly/meshes/Left_S3.stl scale=1 1 1; visual mesh filename=package://assembly/meshes/Left_S3.stl scale=1 1 1
- link left_w0: geometry collision mesh filename=package://assembly/meshes/Left_W0.stl scale=1 1 1; visual mesh filename=package://assembly/meshes/Left_W0.stl scale=1 1 1
- link left_w1: geometry collision mesh filename=package://assembly/meshes/Left_W1.stl scale=1 1 1; visual mesh filename=package://assembly/meshes/Left_W1.stl scale=1 1 1
- link left_w2: geometry collision mesh filename=package://assembly/meshes/Left_W2.stl scale=1 1 1; visual mesh filename=package://assembly/meshes/Left_W2.stl scale=1 1 1
- link right_e1: geometry collision mesh filename=package://assembly/meshes/Right_E1.stl scale=1 1 1; visual mesh filename=package://assembly/meshes/Right_E1.stl scale=1 1 1
- link right_e2: geometry collision mesh filename=package://assembly/meshes/Right_E2.stl scale=1 1 1; visual mesh filename=package://assembly/meshes/Right_E2.stl scale=1 1 1
- link right_gripper: geometry collision mesh filename=package://assembly/meshes/Right_Gripper.stl scale=1 1 1; visual mesh filename=package://assembly/meshes/Right_Gripper.stl scale=1 1 1
- link right_s2: geometry collision mesh filename=package://assembly/meshes/Right_S2.stl scale=1 1 1; visual mesh filename=package://assembly/meshes/Right_S2.stl scale=1 1 1
- link right_s3: geometry collision mesh filename=package://assembly/meshes/Right_S3.stl scale=1 1 1; visual mesh filename=package://assembly/meshes/Right_S3.stl scale=1 1 1
- link right_w0: geometry collision mesh filename=package://assembly/meshes/Right_W0.stl scale=1 1 1; visual mesh filename=package://assembly/meshes/Right_W0.stl scale=1 1 1
- link right_w1: geometry collision mesh filename=package://assembly/meshes/Right_W1.stl scale=1 1 1; visual mesh filename=package://assembly/meshes/Right_W1.stl scale=1 1 1
- link right_w2: geometry collision mesh filename=package://assembly/meshes/Right_W2.stl scale=1 1 1; visual mesh filename=package://assembly/meshes/Right_W2.stl scale=1 1 1
- link s1: geometry collision mesh filename=package://assembly/meshes/S1.stl scale=1 1 1; visual mesh filename=package://assembly/meshes/S1.stl scale=1 1 1
