Commit message: add piper retargeting

File: assets/piper/piper.urdf (robot description, URDF)
Before this commit: robot dual_piper_description, 19 links, 18 joints
Joints:
- joint world_to_der_base: origin xyz=0 -0.3 0 rpy=0 0 0 -> xyz=0 -0.35 0 rpy=0 0 0
- joint world_to_izq_base: origin xyz=0 0.3 0 rpy=0 0 0 -> xyz=0 0.35 0 rpy=0 0 0

Commit message: feat: adding improved piper urdf

File: assets/piper/piper.urdf (robot description, URDF)
Before this commit: robot dual_piper_description, 19 links, 18 joints
Links:
- removed link base_derecho
- removed link base_izquierdo
- removed link der_link1
- removed link der_link2
- removed link der_link3
- removed link der_link4
- removed link der_link5
- removed link der_link6
- removed link der_link7
- removed link der_link8
- removed link izq_link1
- removed link izq_link2
- removed link izq_link3
- removed link izq_link4
- removed link izq_link5
- removed link izq_link6
- removed link izq_link7
- removed link izq_link8
- added link left_base_link, mass 1.02; collision mesh filename=meshes/base_link.STL; visual mesh filename=meshes/base_link.STL
- added link left_dummy_link
- added link left_gripper_base, mass 0.45; collision mesh filename=meshes/gripper_base.STL; visual mesh filename=meshes/gripper_base.STL
- added link left_link1, mass 0.71; collision mesh filename=meshes/link1.STL; visual mesh filename=meshes/link1.STL
- added link left_link2, mass 1.17; collision mesh filename=meshes/link2.STL; visual mesh filename=meshes/link2.STL
- added link left_link3, mass 0.5; collision mesh filename=meshes/link3.STL; visual mesh filename=meshes/link3.STL
- added link left_link4, mass 0.38; collision mesh filename=meshes/link4.STL; visual mesh filename=meshes/link4.STL
- added link left_link5, mass 0.383; collision mesh filename=meshes/link5.STL; visual mesh filename=meshes/link5.STL
- added link left_link6, mass 0.007; collision mesh filename=meshes/link6.STL; visual mesh filename=meshes/link6.STL
- added link left_link7, mass 0.025; collision mesh filename=meshes/link7.STL; visual mesh filename=meshes/link7.STL
- added link left_link8, mass 0.025; collision mesh filename=meshes/link8.STL; visual mesh filename=meshes/link8.STL
- added link right_base_link, mass 1.02; collision mesh filename=meshes/base_link.STL; visual mesh filename=meshes/base_link.STL
- added link right_dummy_link
- added link right_gripper_base, mass 0.45; collision mesh filename=meshes/gripper_base.STL; visual mesh filename=meshes/gripper_base.STL
- added link right_link1, mass 0.71; collision mesh filename=meshes/link1.STL; visual mesh filename=meshes/link1.STL
- added link right_link2, mass 1.17; collision mesh filename=meshes/link2.STL; visual mesh filename=meshes/link2.STL
- added link right_link3, mass 0.5; collision mesh filename=meshes/link3.STL; visual mesh filename=meshes/link3.STL
- added link right_link4, mass 0.38; collision mesh filename=meshes/link4.STL; visual mesh filename=meshes/link4.STL
- added link right_link5, mass 0.383; collision mesh filename=meshes/link5.STL; visual mesh filename=meshes/link5.STL
- added link right_link6, mass 0.007; collision mesh filename=meshes/link6.STL; visual mesh filename=meshes/link6.STL
- added link right_link7, mass 0.025; collision mesh filename=meshes/link7.STL; visual mesh filename=meshes/link7.STL
- added link right_link8, mass 0.025; collision mesh filename=meshes/link8.STL; visual mesh filename=meshes/link8.STL
Joints:
- removed joint der_joint1
- removed joint der_joint2
- removed joint der_joint3
- removed joint der_joint4
- removed joint der_joint5
- removed joint der_joint6
- removed joint der_joint7
- removed joint der_joint8
- removed joint izq_joint1
- removed joint izq_joint2
- removed joint izq_joint3
- removed joint izq_joint4
- removed joint izq_joint5
- removed joint izq_joint6
- removed joint izq_joint7
- removed joint izq_joint8
- removed joint world_to_der_base
- removed joint world_to_izq_base
- added joint left_base_to_dummy: type fixed, parent left_dummy_link, child left_base_link, origin xyz=0 0 0 rpy=0 0 0
- added joint left_joint1: type revolute, parent left_base_link, child left_link1, origin xyz=0 0 0.123 rpy=0 0 0, axis 0 0 1, limit lower=-2.618 upper=2.618 effort=100 velocity=5
- added joint left_joint2: type revolute, parent left_link1, child left_link2, origin xyz=0 0 0 rpy=1.5708 -0.1359 -3.1416, axis 0 0 1, limit lower=0 upper=3.14 effort=100 velocity=5
- added joint left_joint3: type revolute, parent left_link2, child left_link3, origin xyz=0.28503 0 0 rpy=0 0 -1.7939, axis 0 0 1, limit lower=-2.967 upper=0 effort=100 velocity=5
- added joint left_joint4: type revolute, parent left_link3, child left_link4, origin xyz=-0.021984 -0.25075 0 rpy=1.5708 0 0, axis 0 0 1, limit lower=-1.745 upper=1.745 effort=100 velocity=5
- added joint left_joint5: type revolute, parent left_link4, child left_link5, origin xyz=0 0 0 rpy=-1.5708 0 0, axis 0 0 1, limit lower=-1.22 upper=1.22 effort=100 velocity=5
- added joint left_joint6: type revolute, parent left_link5, child left_link6, origin xyz=8.8259E-05 -0.091 0 rpy=1.5708 0 0, axis 0 0 1, limit lower=-2.0944 upper=2.0944 effort=100 velocity=3
- added joint left_joint6_to_gripper_base: type fixed, parent left_link6, child left_gripper_base, origin xyz=0 0 0 rpy=0 0 0
- added joint left_joint7: type prismatic, parent left_gripper_base, child left_link7, origin xyz=0 0 0.1358 rpy=1.5708 0 0, axis 0 0 1, limit lower=0 upper=0.035 effort=10 velocity=1
- added joint left_joint8: type prismatic, parent left_gripper_base, child left_link8, origin xyz=0 0 0.1358 rpy=1.5708 0 -3.1416, axis 0 0 -1, limit lower=-0.035 upper=0 effort=10 velocity=1
- added joint right_base_to_dummy: type fixed, parent right_dummy_link, child right_base_link, origin xyz=0 0 0 rpy=0 0 0
- added joint right_joint1: type revolute, parent right_base_link, child right_link1, origin xyz=0 0 0.123 rpy=0 0 0, axis 0 0 1, limit lower=-2.618 upper=2.618 effort=100 velocity=5
- added joint right_joint2: type revolute, parent right_link1, child right_link2, origin xyz=0 0 0 rpy=1.5708 -0.1359 -3.1416, axis 0 0 1, limit lower=0 upper=3.14 effort=100 velocity=5
- added joint right_joint3: type revolute, parent right_link2, child right_link3, origin xyz=0.28503 0 0 rpy=0 0 -1.7939, axis 0 0 1, limit lower=-2.967 upper=0 effort=100 velocity=5
- added joint right_joint4: type revolute, parent right_link3, child right_link4, origin xyz=-0.021984 -0.25075 0 rpy=1.5708 0 0, axis 0 0 1, limit lower=-1.745 upper=1.745 effort=100 velocity=5
- added joint right_joint5: type revolute, parent right_link4, child right_link5, origin xyz=0 0 0 rpy=-1.5708 0 0, axis 0 0 1, limit lower=-1.22 upper=1.22 effort=100 velocity=5
- added joint right_joint6: type revolute, parent right_link5, child right_link6, origin xyz=8.8259E-05 -0.091 0 rpy=1.5708 0 0, axis 0 0 1, limit lower=-2.0944 upper=2.0944 effort=100 velocity=3
- added joint right_joint6_to_gripper_base: type fixed, parent right_link6, child right_gripper_base, origin xyz=0 0 0 rpy=0 0 0
- added joint right_joint7: type prismatic, parent right_gripper_base, child right_link7, origin xyz=0 0 0.1358 rpy=1.5708 0 0, axis 0 0 1, limit lower=0 upper=0.035 effort=10 velocity=1
- added joint right_joint8: type prismatic, parent right_gripper_base, child right_link8, origin xyz=0 0 0.1358 rpy=1.5708 0 -3.1416, axis 0 0 -1, limit lower=-0.035 upper=0 effort=10 velocity=1
- added joint world_to_left: type fixed, parent world, child left_dummy_link, origin xyz=0.0 0.3 0.0 rpy=0 0 0
- added joint world_to_right: type fixed, parent world, child right_dummy_link, origin xyz=0.0 -0.3 0.0 rpy=0 0 0
