Commit message: fix(piper): mount the bimanual bases 60 cm apart
What changed:
- The URDF and MJCF placed the arms at +/-0.35 m; the physical BiPiper is
  mounted 0.60 m apart, which is also the repo-wide bimanual convention. Both
  files move together so the kinematic and simulation models cannot drift.
- tblock episode 0 improves with the corrected geometry: 0.13 cm mean / 0.28 cm
  max TCP error against 0.14 / 0.35, still collision-free, still --strict-ik.
- The table stays laterally centered. A sideways offset does rescue individual
  episodes that fold one arm, but distorting a shared calibration for one
  recording is worse than dropping that recording; screening handles those.
- test_sim_profile_is_separate_from_lab_config compared against hard-coded
  table coordinates, so every placement re-fit broke an unrelated test. It now
  reads the shipped file and asserts what it is actually about: that the lab
  calibration was not selected.

Verification:
- `handumi replay outputs/datasets/tblock --robot piper --strict-ik` — passed
- `pytest` — 100 passed, 1 pre-existing failure unrelated to this change

File: assets/piper/piper.urdf (robot description, URDF)
Before this commit: robot dual_piper, 25 links, 24 joints
Joints:
- joint world_to_left: origin xyz=0.0 0.35 0.0 rpy=0 0 0 -> xyz=0.0 0.30 0.0 rpy=0 0 0
- joint world_to_right: origin xyz=0.0 -0.35 0.0 rpy=0 0 0 -> xyz=0.0 -0.30 0.0 rpy=0 0 0

Commit message: fix(piper): place the URDF TCP on the gripper fingertip plane
What changed:
- assets/piper/piper.urdf moves left_tcp/right_tcp from 0.145 m to 0.1358 m
  along link6 z. The official piper_description meshes (byte-identical to
  ours) put the finger joints and the end of the finger pads at 0.1358 m; the
  0.145 came from our solver v0.1 and sat 9 mm past the fingers, so IK left
  the real tips 9 mm short of the demonstrated HandUMI tip. AgileX publishes
  no TCP frame of its own.
- Measured on tblock after reconversion (v4): fingertip minimum height over
  the table now matches the demonstration (p50 1.38 cm vs 2.08 cm before),
  lower in 172 of 172 working arms. Every other embodiment is untouched.

Verification:
- `JAX_PLATFORMS=cpu uv run pytest tests/robots tests/dataset/test_screening.py -q` — 43 passed
- `JAX_PLATFORMS=cpu uv run pytest tests -q --ignore=tests/real` — 251 passed

File: assets/piper/piper.urdf (robot description, URDF)
Before this commit: robot dual_piper, 25 links, 24 joints
Joints:
- joint left_link6_to_tcp: origin xyz=0 0 0.145 rpy=0 0 0 -> xyz=0 0 0.1358 rpy=0 0 0
- joint right_link6_to_tcp: origin xyz=0 0 0.145 rpy=0 0 0 -> xyz=0 0 0.1358 rpy=0 0 0
