Commit message: fix(piper): match 0.68 m bimanual spacing and left home_q
What changed:
- URDF/MuJoCo base offsets at ±0.34 m to match the physical BiPiper mount
- Left arm home_q elbow matches the right; drop redundant world_collision_plane_z

Verification:
- `uv run pytest tests/robots/test_registry.py -q` — passed (prior run)

Co-authored-by: Cursor <cursoragent@cursor.com>

File: assets/piper/piper.urdf (robot description, URDF)
Before this commit: robot dual_piper, 25 links, 24 joints
Joints:
- joint world_to_left: origin xyz=0.0 0.30 0.0 rpy=0 0 0 -> xyz=0.0 0.34 0.0 rpy=0 0 0
- joint world_to_right: origin xyz=0.0 -0.30 0.0 rpy=0 0 0 -> xyz=0.0 -0.34 0.0 rpy=0 0 0
