Commit message: feat(robots): add opt-in capsule collision avoidance to bimanual IK
What changed:
- KinematicsConfig gains self/world collision weights, margins, the tabletop
  plane height, and a pair-scope switch; with both weights at 0 the solver
  keeps the exact legacy cost structure and compiled cache, so only robots
  whose YAML opts in change behavior.
- registry builds the capsule model once per embodiment and prunes pairs that
  are unavoidable rather than faults: structural overlaps at home_q (MoveIt's
  generated-disable-list idea) and same-gripper assemblies, since fingers
  closing on each other is grasping.
- A jitted two-tier proximity gate picks the cheapest solve variant per frame,
  keeping the metal replay at ~16 ms/frame instead of ~95 ms.

Verification:
- `pytest tests/robots/test_registry.py` (staged snapshot, isolated worktree) — 12 passed
- `handumi replay outputs/datasets/tblock --robot metal` — audit over 320 frames shows no actionable interpenetration

File: assets/metal/metal_bimanual.urdf (robot description, URDF)
Before this commit: robot metal_bimanual, 25 links, 24 joints
Links:
- link left_base_link: geometry collision mesh filename=meshes/base_link.STL; visual mesh filename=meshes/base_link.STL
- link left_gripper_base: geometry collision mesh filename=meshes/gripper_base.STL; visual mesh filename=meshes/gripper_base.STL
- link left_link1: geometry collision mesh filename=meshes/link1.STL; visual mesh filename=meshes/link1.STL
- link left_link2: geometry collision mesh filename=meshes/link2.STL; visual mesh filename=meshes/link2.STL
- link left_link3: geometry collision mesh filename=meshes/link3.STL; visual mesh filename=meshes/link3.STL
- link left_link4: geometry collision mesh filename=meshes/link4.STL; visual mesh filename=meshes/link4.STL
- link left_link5: geometry collision mesh filename=meshes/link5.STL; visual mesh filename=meshes/link5.STL
- link left_link6: geometry collision mesh filename=meshes/link6.STL; visual mesh filename=meshes/link6.STL
- link left_link7: geometry collision mesh filename=meshes/link7.STL; visual mesh filename=meshes/link7.STL
- link left_link8: geometry collision mesh filename=meshes/link8.STL; visual mesh filename=meshes/link8.STL
- link right_base_link: geometry collision mesh filename=meshes/base_link.STL; visual mesh filename=meshes/base_link.STL
- link right_gripper_base: geometry collision mesh filename=meshes/gripper_base.STL; visual mesh filename=meshes/gripper_base.STL
- link right_link1: geometry collision mesh filename=meshes/link1.STL; visual mesh filename=meshes/link1.STL
- link right_link2: geometry collision mesh filename=meshes/link2.STL; visual mesh filename=meshes/link2.STL
- link right_link3: geometry collision mesh filename=meshes/link3.STL; visual mesh filename=meshes/link3.STL
- link right_link4: geometry collision mesh filename=meshes/link4.STL; visual mesh filename=meshes/link4.STL
- link right_link5: geometry collision mesh filename=meshes/link5.STL; visual mesh filename=meshes/link5.STL
- link right_link6: geometry collision mesh filename=meshes/link6.STL; visual mesh filename=meshes/link6.STL
- link right_link7: geometry collision mesh filename=meshes/link7.STL; visual mesh filename=meshes/link7.STL
- link right_link8: geometry collision mesh filename=meshes/link8.STL; visual mesh filename=meshes/link8.STL
