Commit message: fix(r1lite): target the fingertip TCP and open the mirrored finger
What changed:
- assets/r1lite/r1lite.urdf: add left_tcp/right_tcp at the fingertip plane,
  0.0784 m ahead of the gripper link, and use the production dark/silver
  finish instead of the CAD's orange and blue
- configs/robots/r1lite.yaml: IK targets the new TCPs; finger_joint2 opens to
  -0.05, inside its mirrored [-0.05, 0] URDF range, also in home_q

Verification:
- `uv run pytest -q tests/robots tests/scripts` — passed (70 passed, 2 skipped)
- home_q within URDF limits after the sign fix

File: assets/r1lite/r1lite.urdf (robot description, URDF)
Before this commit: robot r1lite, 34 links, 33 joints
Links:
- added link left_tcp
- added link right_tcp
Joints:
- added joint left_gripper_to_tcp: type fixed, parent left_gripper_link, child left_tcp, origin xyz=0.0784 0 0 rpy=0 0 0
- added joint right_gripper_to_tcp: type fixed, parent right_gripper_link, child right_tcp, origin xyz=0.0784 0 0 rpy=0 0 0
